Commit message: Limited ROM

File: static/urdf/skeleton.urdf (robot description, URDF)
Before this commit: robot both_arm_baymax_skeleton, 10 links, 9 joints
Joints:
- joint left_elbow_joint: limit lower=-1.57 upper=0.0 effort=100 velocity=10 -> lower=-0.785 upper=0.0 effort=100 velocity=10
- joint right_elbow_joint: limit lower=0.0 upper=1.57 effort=100 velocity=10 -> lower=0.0 upper=0.785 effort=100 velocity=10
